File: kicad/ampermeter/ampermeter.sch (KiCad schematic (older format))
At the start: 56 parts, among them J1 SWD, J2 USB_B_Micro, J3 UART, J4 ILI_9321(2.2inch), SW1 PowerOn, SW2 EVQWKL001, U1 ISL9204, U2 TPS60241DGKR, U3 HT7333, U4 STM32H750VITx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

Commit message: - изначальный коммит кода
Parts:
- R10, R11, R12, R7, R8, R9: value 33 -> 300
Connections:
- wire segments 202 -> 205
Other:
- note added: "PE13-PE14 соединенны перемычкой впоследствии"
Changed lines of the file:
@@
 U 1 1 5D994A07
 P 2600 5750
-F 0 "R12" V 2550 5900 50  0000 C CNN
-F 1 "33" V 2600 5750 50  0000 C CNN
+F 0 "R12" V 2550 5950 50  0000 C CNN
+F 1 "300" V 2600 5750 50  0000 C CNN
 F 2 "Resistor_SMD:R_0603_1608Metric" V 2530 5750 50  0001 C CNN
 F 3 "~" H 2600 5750 50  0001 C CNN
@@
 U 1 1 5D9A5C48
 P 2600 5650
-F 0 "R11" V 2550 5800 50  0000 C CNN
-F 1 "33" V 2600 5650 50  0000 C CNN
+F 0 "R11" V 2550 5850 50  0000 C CNN
+F 1 "300" V 2600 5650 50  0000 C CNN
 F 2 "Resistor_SMD:R_0603_1608Metric" V 2530 5650 50  0001 C CNN
 F 3 "~" H 2600 5650 50  0001 C CNN
@@
 P 4900 4350
 F 0 "R7" V 4850 4500 50  0000 C CNN
-F 1 "33" V 4900 4350 50  0000 C CNN
+F 1 "300" V 4900 4350 50  0000 C CNN
 F 2 "Resistor_SMD:R_0603_1608Metric" V 4830 4350 50  0001 C CNN
 F 3 "~" H 4900 4350 50  0001 C CNN
@@
 P 4900 4450
 F 0 "R8" V 4850 4600 50  0000 C CNN
-F 1 "33" V 4900 4450 50  0000 C CNN
+F 1 "300" V 4900 4450 50  0000 C CNN
 F 2 "Resistor_SMD:R_0603_1608Metric" V 4830 4450 50  0001 C CNN
 F 3 "~" H 4900 4450 50  0001 C CNN
@@
 P 4900 4550
 F 0 "R9" V 4850 4700 50  0000 C CNN
-F 1 "33" V 4900 4550 50  0000 C CNN
+F 1 "300" V 4900 4550 50  0000 C CNN
 F 2 "Resistor_SMD:R_0603_1608Metric" V 4830 4550 50  0001 C CNN
 F 3 "~" H 4900 4550 50  0001 C CNN
@@
 P 4900 4650
 F 0 "R10" V 4850 4800 50  0000 C CNN
-F 1 "33" V 4900 4650 50  0000 C CNN
+F 1 "300" V 4900 4650 50  0000 C CNN
 F 2 "Resistor_SMD:R_0603_1608Metric" V 4830 4650 50  0001 C CNN
 F 3 "~" H 4900 4650 50  0001 C CNN
@@
 	2850 4350 2700 4350
 Wire Wire Line
-	2850 4550 2700 4550
+	2850 4550 2800 4550
 Text Notes 4800 4800 0    50   ~ 0
 R7-R12 попробуем 300 Ом
+Wire Wire Line
+	2850 4450 2800 4450
+Wire Wire Line
+	2800 4450 2800 4550
+Connection ~ 2800 4550
+Wire Wire Line
+	2800 4550 2700 4550
+Text Notes 750  4750 0    50   ~ 0
+PE13-PE14 соединенны перемычкой впоследствии
 $EndSCHEMATC
