File: kicad/ampermeter/analog.sch (KiCad schematic (older format))
At the start: 56 parts, among them J5 Vout, J6 Isense, J7 GND, Q1 SI2302, Q2 SI2302, Q3 IRLML2502, U10 ADS1251, U6 LM4140, U7 TPS79301-EP, U8 AD8031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

Commit message: - изначальный коммит кода
Parts:
- R24, R25: value 10k -> inf
- R26, R28: value 5.1k -> 30
Changed lines of the file:
@@
 P 7200 3150
 F 0 "R26" V 7300 3150 50  0000 C CNN
-F 1 "5.1k" V 7200 3150 50  0000 C CNN
+F 1 "30" V 7200 3150 50  0000 C CNN
 F 2 "Resistor_SMD:R_0603_1608Metric" V 7130 3150 50  0001 C CNN
 F 3 "~" H 7200 3150 50  0001 C CNN
@@
 P 7200 3350
 F 0 "R28" V 7300 3350 50  0000 C CNN
-F 1 "5.1k" V 7200 3350 50  0000 C CNN
+F 1 "30" V 7200 3350 50  0000 C CNN
 F 2 "Resistor_SMD:R_0603_1608Metric" V 7130 3350 50  0001 C CNN
 F 3 "~" H 7200 3350 50  0001 C CNN
@@
 P 7400 2950
 F 0 "R24" V 7500 2950 50  0000 C CNN
-F 1 "10k" V 7400 2950 50  0000 C CNN
+F 1 "inf" V 7400 2950 50  0000 C CNN
 F 2 "Resistor_SMD:R_0603_1608Metric" V 7330 2950 50  0001 C CNN
 F 3 "~" H 7400 2950 50  0001 C CNN
@@
 P 7600 2950
 F 0 "R25" V 7700 2950 50  0000 C CNN
-F 1 "10k" V 7600 2950 50  0000 C CNN
+F 1 "inf" V 7600 2950 50  0000 C CNN
 F 2 "Resistor_SMD:R_0603_1608Metric" V 7530 2950 50  0001 C CNN
 F 3 "~" H 7600 2950 50  0001 C CNN
