File: kicad/isolated_usb2uart/isolated_usb2uart.sch (KiCad schematic (older format))
At the start: 14 parts, among them J1 Conn_01x04, J2 USB_B_Micro, U1 ISO7221BDR, U2 FT230XQ

Commit message: - изначальный коммит кода
Parts:
- J2: symbol Connector:USB_B_Micro -> isolated_usb2uart-rescue:USB_B_Micro-Connector
Changed lines of the file:
@@
 $EndDescr
 $Comp
-L Connector:USB_B_Micro J2
+L isolated_usb2uart-rescue:USB_B_Micro-Connector J2
 U 1 1 5D907AF4
 P 2850 2750
