File: kicad/ADS1271/ADS1271.sch (KiCad schematic (older format))
At the start: 85 parts, among them J1 ADC_IN, J2 Data&Power, J3 Conn_01x02, U1 AD8628, U10 LM4140-2.5V, U11 MCP1700-3302E_SOT23, U12 TPS60241DGKR, U13 TPS60241DGKR, U2 AD8628, U3 AD8628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

Commit message: - получили какие-то разумные цифры с аналоговой части
Other:
- note added: "Vin = +-100 mV"
- note added: "Временно перепаяем U9 на 2.0V (было 2.5V)\nРезисторы R7, R18 увеличим до 3 KOm (было 1.5 КОм)\nКУ=10 (было КУ=19)"
Changed lines of the file:
@@
 Text Notes 1800 850  0    50   ~ 0
 BAV - задом наперед черт побери!!!!
+Text Notes 3500 2200 0    50   ~ 0
+Vin = +-100 mV
+Text Notes 1350 4000 0    50   ~ 0
+Временно перепаяем U9 на 2.0V (было 2.5V)\nРезисторы R7, R18 увеличим до 3 KOm (было 1.5 КОм)\nКУ=10 (было КУ=19)
 $EndSCHEMATC
