File: kicad/stm32h7_digital/stm32h7_digital.sch (KiCad schematic (older format))
At the start: 39 parts, among them J1 SWD, J2 USB_B_Micro, J3 UART, J4 PA0-7, J5 SPI3, J6 Data&Power, J7 Display, SW1 PowerOn, SW2 EVQWKL001, U1 ISL9204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

Commit message: - попробовали писать во flash за пределы первой страницы (неудачно)
- запаяли qspi flash и заставили её работать в spi режиме
Other:
- note added: "~QSPI_CS - нужно к PC11 прицеплять"
Changed lines of the file:
@@
 Wire Wire Line
 	8950 900  8950 850
+Text Notes 9000 3750 0    50   ~ 0
+~QSPI_CS - нужно к PC11 прицеплять
 $EndSCHEMATC
