File: kicad/analog_frontend/analog_frontend.sch (KiCad schematic (older format))
At the start: 35 parts, among them J1 Power, J2 Vout, J3 ADC, J4 Isense, J5 GND, J6 Digital, Q1 SI2302, Q2 SI2302, Q3 IRLML2502, U1 TPS79301-EP

Commit message: - получили какие-то разумные цифры с аналоговой части
Parts:
- C3: value 1n -> 100p
- C5: value 25u -> 10u
- R1: value 2k -> 27k
- R10, R11, R12: value 4.7k -> 1k
- R4: value 2k -> 750
- R9: value 1 -> 1.2
Other:
- note added: "+-130 mV"
- note added: "R6, R7, R8, R9 желательно точные резисторы"
Changed lines of the file:
@@
 P 3750 1650
 F 0 "C5" H 3865 1696 50  0000 L CNN
-F 1 "25u" H 3865 1605 50  0000 L CNN
+F 1 "10u" H 3865 1605 50  0000 L CNN
 F 2 "Capacitor_SMD:C_1206_3216Metric" H 3788 1500 50  0001 C CNN
 F 3 "~" H 3750 1650 50  0001 C CNN
@@
 P 4200 1250
 F 0 "R1" V 4300 1250 50  0000 C CNN
-F 1 "2k" V 4200 1250 50  0000 C CNN
+F 1 "27k" V 4200 1250 50  0000 C CNN
 F 2 "Resistor_SMD:R_0603_1608Metric" V 4130 1250 50  0001 C CNN
 F 3 "~" H 4200 1250 50  0001 C CNN
@@
 P 4200 1600
 F 0 "R4" V 4300 1600 50  0000 C CNN
-F 1 "2k" V 4200 1600 50  0000 C CNN
+F 1 "750" V 4200 1600 50  0000 C CNN
 F 2 "Resistor_SMD:R_0603_1608Metric" V 4130 1600 50  0001 C CNN
 F 3 "~" H 4200 1600 50  0001 C CNN
@@
 P 4450 1600
 F 0 "C3" H 4565 1646 50  0000 L CNN
-F 1 "1n" H 4565 1555 50  0000 L CNN
+F 1 "100p" H 4565 1555 50  0000 L CNN
 F 2 "Capacitor_SMD:C_0603_1608Metric" H 4488 1450 50  0001 C CNN
 F 3 "~" H 4450 1600 50  0001 C CNN
@@
 P 3650 3450
 F 0 "R9" V 3750 3450 50  0000 C CNN
-F 1 "1" V 3650 3450 50  0000 C CNN
+F 1 "1.2" V 3650 3450 50  0000 C CNN
 F 2 "Resistor_SMD:R_0805_2012Metric" V 3580 3450 50  0001 C CNN
 F 3 "~" H 3650 3450 50  0001 C CNN
@@
 P 2450 3650
 F 0 "R11" V 2550 3650 50  0000 C CNN
-F 1 "4.7k" V 2450 3650 50  0000 C CNN
+F 1 "1k" V 2450 3650 50  0000 C CNN
 F 2 "Resistor_SMD:R_0603_1608Metric" V 2380 3650 50  0001 C CNN
 F 3 "~" H 2450 3650 50  0001 C CNN
@@
 P 3300 3650
 F 0 "R12" V 3400 3650 50  0000 C CNN
-F 1 "4.7k" V 3300 3650 50  0000 C CNN
+F 1 "1k" V 3300 3650 50  0000 C CNN
 F 2 "Resistor_SMD:R_0603_1608Metric" V 3230 3650 50  0001 C CNN
 F 3 "~" H 3300 3650 50  0001 C CNN
@@
 P 1600 3650
 F 0 "R10" V 1700 3650 50  0000 C CNN
-F 1 "4.7k" V 1600 3650 50  0000 C CNN
+F 1 "1k" V 1600 3650 50  0000 C CNN
 F 2 "Resistor_SMD:R_0603_1608Metric" V 1530 3650 50  0001 C CNN
 F 3 "~" H 1600 3650 50  0001 C CNN
@@
 	1    0    0    -1
 $EndComp
+Text Notes 6600 2350 0    50   ~ 0
++-130 mV
+Text Notes 2300 3200 0    50   ~ 0
+R6, R7, R8, R9 желательно точные резисторы
 $EndSCHEMATC

Commit message: - sch info text
Parts:
- C6, C7, C8: value 22n -> 100
Changed lines of the file:
@@
-	1    0    0    -1
-$EndComp
-$Comp
-L Device:C C6
-U 1 1 5FC1A941
-P 1500 4300
-F 0 "C6" H 1615 4346 50  0000 L CNN
-F 1 "22n" H 1615 4255 50  0000 L CNN
-F 2 "Capacitor_SMD:C_0603_1608Metric" H 1538 4150 50  0001 C CNN
-F 3 "~" H 1500 4300 50  0001 C CNN
-	1    1500 4300
-	1    0    0    -1
-$EndComp
-$Comp
-L Device:C C7
-U 1 1 5FC1A947
-P 2350 4300
-F 0 "C7" H 2465 4346 50  0000 L CNN
-F 1 "22n" H 2465 4255 50  0000 L CNN
-F 2 "Capacitor_SMD:C_0603_1608Metric" H 2388 4150 50  0001 C CNN
-F 3 "~" H 2350 4300 50  0001 C CNN
-	1    2350 4300
-	1    0    0    -1
-$EndComp
-$Comp
-L Device:C C8
-U 1 1 5FC1A94D
-P 3200 4300
-F 0 "C8" H 3315 4346 50  0000 L CNN
-F 1 "22n" H 3315 4255 50  0000 L CNN
-F 2 "Capacitor_SMD:C_0603_1608Metric" H 3238 4150 50  0001 C CNN
-F 3 "~" H 3200 4300 50  0001 C CNN
-	1    3200 4300
 	1    0    0    -1
 $EndComp
 Wire Wire Line
 	3300 3800 3200 3800
-Wire Wire Line
-	3200 3800 3200 4150
 Wire Wire Line
 	2450 3800 2350 3800
@@
 F 3 "" H 2350 4450 50  0001 C CNN
 	1    2350 4450
-	1    0    0    -1
-$EndComp
-$Comp
-L power:GND #PWR021
-U 1 1 5FC1A965
-P 3200 4450
-F 0 "#PWR021" H 3200 4200 50  0001 C CNN
-F 1 "GND" H 3205 4277 50  0001 C CNN
-F 2 "" H 3200 4450 50  0001 C CNN
-F 3 "" H 3200 4450 50  0001 C CNN
-	1    3200 4450
 	1    0    0    -1
 $EndComp
@@
 Text Notes 2300 3200 0    50   ~ 0
 R6, R7, R8, R9 желательно точные резисторы
+Wire Wire Line
+	3200 3800 3200 4150
+$Comp
+L power:GND #PWR021
+U 1 1 5FC1A965
+P 3200 4450
+F 0 "#PWR021" H 3200 4200 50  0001 C CNN
+F 1 "GND" H 3205 4277 50  0001 C CNN
+F 2 "" H 3200 4450 50  0001 C CNN
+F 3 "" H 3200 4450 50  0001 C CNN
+	1    3200 4450
+	1    0    0    -1
+$EndComp
+$Comp
+L Device:C C8
+U 1 1 5FC1A94D
+P 3200 4300
+F 0 "C8" H 3315 4346 50  0000 L CNN
+F 1 "100" H 3315 4255 50  0000 L CNN
+F 2 "Capacitor_SMD:C_0603_1608Metric" H 3238 4150 50  0001 C CNN
+F 3 "~" H 3200 4300 50  0001 C CNN
+	1    3200 4300
+	1    0    0    -1
+$EndComp
+$Comp
+L Device:C C7
+U 1 1 5FC1A947
+P 2350 4300
+F 0 "C7" H 2465 4346 50  0000 L CNN
+F 1 "100" H 2465 4255 50  0000 L CNN
+F 2 "Capacitor_SMD:C_0603_1608Metric" H 2388 4150 50  0001 C CNN
+F 3 "~" H 2350 4300 50  0001 C CNN
+	1    2350 4300
+	1    0    0    -1
+$EndComp
+$Comp
+L Device:C C6
+U 1 1 5FC1A941
+P 1500 4300
+F 0 "C6" H 1615 4346 50  0000 L CNN
+F 1 "100" H 1615 4255 50  0000 L CNN
+F 2 "Capacitor_SMD:C_0603_1608Metric" H 1538 4150 50  0001 C CNN
+F 3 "~" H 1500 4300 50  0001 C CNN
+	1    1500 4300
+	1    0    0    -1
+$EndComp
 $EndSCHEMATC
